File: elect.brd (EAGLE design)
At the start: 250 x 120 mm, 2 parts

Commit message: Update elect.brd
Parts:
- removed ACTUATOR1: SERVO01, TinkerTools:SG90
- removed ACTUATOR2: SERVO02, TinkerTools:SG90
- added SERVO1, SERVO2, SERVO3, SERVO4: SERVOSG90, Tinkercad:SG90
- added U1: ARDUINO-UNO-R3-SHIELD, Tinkercad:ARDUINO-UNO-R3-SHIELD
Connections:
- removed net SERVO_SIGNAL_1: ACTUATOR1.1, ACTUATOR2.1
- new net U1_5V: SERVO1.2, SERVO2.2, SERVO3.2, SERVO4.2, U1.5V
- new net U1_D3: SERVO3.3, U1.D3
- new net U1_D5: SERVO1.3, U1.D5
- new net U1_D6: SERVO2.3, U1.D6
- new net U1_D9: SERVO4.3, U1.D9
- new net U1_GND: SERVO1.1, SERVO2.1, SERVO3.1, SERVO4.1, U1.GND@0, U1.GND@1, U1.GND@2
Other:
- board size 250 x 120 mm -> 233.8 x 102.8 mm
